File: usbcan_20190426.brd (EAGLE design)
At the start: 40 x 50 mm, 45 parts, among them J1 8P8C-LED, J2 MICRO-USB-RECEPTACLE47589-0001, J3 MA04-1, J4 MA02-2, U1 STM32F302C, U2 NCV7351D1E, U3 SI8621AB-B-IS, U4 AP2127N-3.3TRG1, U5 78L05F, X1 CSTCE8M00G55

Commit message: brdのbootとgndをつなげた1
Connections:
- net GNDA: now also U1.44
